Commit message: Added coverage test

File: simulation_ws/src/cr2_description/params/cr2_params.urdf.xacro (robot description, xacro)
@@ -31,4 +31,6 @@
     <!--DEBUG-->
     <!--/DEBUG-->
+    <xacro:property name="body_color"           value="DarkGrey"/>
+    <xacro:property name="back_cover_color"     value="DarkGrey"/>
 <!--BODY-->
     <!--TODO measure on assambled robot-->

File: simulation_ws/src/cr2_description/robot/cr2.gazebo.xacro (robot description, xacro)
@@ -4,24 +4,23 @@
         name="cr2">
   <gazebo>
-  <plugin name="gazebo_ros_control" filename="libgazebo_ros_control.so">
-    <robotNamespace>/</robotNamespace>
-    <legacyModeNS>true</legacyModeNS>
-  </plugin>
-  <plugin name="ridgeback_ros_force_based_move"
-          filename="libridgeback_ros_force_based_move.so">
-    <robotNamespace>/</robotNamespace>
-    <commandTopic>cmd_vel</commandTopic>
-    <odometryTopic>odom</odometryTopic>
-    <odometryFrame>odom</odometryFrame>
-    <odometryRate>25.0</odometryRate>
-    <robotBaseFrame>base_link</robotBaseFrame>
-    <cmdVelTimeOut>0.25</cmdVelTimeOut>
-    <!-- Don't publish a transform: the controller does it. -->
-    <publishOdometryTf>0.0</publishOdometryTf>
-    <yaw_velocity_p_gain>500.0</yaw_velocity_p_gain>
-    <x_velocity_p_gain>10000.0</x_velocity_p_gain>
-    <y_velocity_p_gain>10000.0</y_velocity_p_gain>
-  </plugin>
- <gazebo>
+    <plugin name="gazebo_ros_control" filename="libgazebo_ros_control.so">
+      <robotNamespace>/</robotNamespace>
+      <legacyModeNS>true</legacyModeNS>
+    </plugin>
+    <plugin name="ridgeback_ros_force_based_move"
+            filename="libridgeback_ros_force_based_move.so">
+      <robotNamespace>/</robotNamespace>
+      <commandTopic>cmd_vel</commandTopic>
+      <odometryTopic>odom</odometryTopic>
+      <odometryFrame>odom</odometryFrame>
+      <odometryRate>25.0</odometryRate>
+      <robotBaseFrame>base_link</robotBaseFrame>
+      <cmdVelTimeOut>0.25</cmdVelTimeOut>
+      <!-- Don't publish a transform: the controller does it. -->
+      <publishOdometryTf>false</publishOdometryTf>
+      <yaw_velocity_p_gain>500.0</yaw_velocity_p_gain>
+      <x_velocity_p_gain>10000.0</x_velocity_p_gain>
+      <y_velocity_p_gain>10000.0</y_velocity_p_gain>
+    </plugin>
     <plugin name="imu_plugin" filename="libgazebo_ros_imu.so">
       <alwaysOn>true</alwaysOn>
@@ -32,5 +31,4 @@
       <updateRate>20.0</updateRate>
     </plugin>
-  </gazebo>
     <!--TODO ALLSO BAD EGG - need more efforts-->
   <!--<plugin name="gazebo_ros_joint_state_publisher" filename="libgazebo_ros_joint_state_publisher.so">-->
@@ -40,4 +38,17 @@
   <!--</plugin>-->
   </gazebo>
+  <gazebo reference="body">
+    <xacro:set_gazebo_material color="DarkGrey"/>
+  </gazebo>
+<!--
+  <gazebo reference="head">
+    <material>Gazebo/DarkGrey</material>
+  </gazebo>
+  <gazebo reference="back_cover">
+    <material>Gazebo/DarkGrey</material>
+  </gazebo>
+  <gazebo reference="tray">
+    <material>Gazebo/DarkGrey</material>
+  </gazebo> -->
   <!-- ///////////////////////-->
   <!-- Mechanum wheels chassis-->
@@ -48,35 +59,6 @@
     <!--<kp value="10000000.0"/>-->
     <!--<kd value="1.0"/>-->
-    <material>Gazebo/White</material>
     <gravity>true</gravity>
   </gazebo>
-  <!--<gazebo reference="FL_wheel_link">-->
-    <!--<mu1 value="0.0"/>-->
-    <!--<mu2 value="0.0"/>-->
-    <!--<kp value="10000000.0"/>-->
-    <!--<kd value="1.0"/>-->
-    <!--<material>Gazebo/Blue</material>-->
-  <!--</gazebo>-->
-  <!--<gazebo reference="FR_wheel_link">-->
-    <!--<mu1 value="0.0"/>-->
-    <!--<mu2 value="0.0"/>-->
-    <!--<kp value="10000000.0"/>-->
-    <!--<kd value="1.0"/>-->
-    <!--<material>Gazebo/Blue</material>-->
-  <!--</gazebo>-->
-  <!--<gazebo reference="RL_wheel_link">-->
-    <!--<mu1 value="0.0"/>-->
-    <!--<mu2 value="0.0"/>-->
-    <!--<kp value="10000000.0"/>-->
-    <!--<kd value="1.0"/>-->
-    <!--<material>Gazebo/Blue</material>-->
-  <!--</gazebo>-->
-  <!--<gazebo reference="RR_wheel_link">-->
-    <!--<mu1 value="0.0"/>-->
-    <!--<mu2 value="0.0"/>-->
-    <!--<kp value="10000000.0"/>-->
-    <!--<kd value="1.0"/>-->
-    <!--<material>Gazebo/Blue</material>-->
-  <!--</gazebo>-->
   <gazebo reference="rear_left_wheel_link">
     <mu1 value="0.0"/>
@@ -270,5 +252,5 @@
   <!---->
   <!--ULTRASONIC-->
-  <!--<xacro:ultrasonic_gazebo position="FRONT_TOP"/>-->
+  <xacro:ultrasonic_gazebo position="FRONT_TOP"/>
   <!--<xacro:ultrasonic_gazebo position="FRONT_BOTTOM"/>-->
   <!--<xacro:ultrasonic_gazebo position="FRONT_BOTTOM_LEFT"/>-->

File: simulation_ws/src/cr2_description/urdf/helpers/add_body.urdf.xacro (robot description, xacro)
@@ -13,5 +13,5 @@
                         mash_filename="${cr2_body_mash}"
                         scale_proportion="${scale_proportion}" />
-                <xacro:red_material/>
+                <xacro:set_material color="${body_color}"/>
                 <xacro:body_to_base_platform_translation_mash/>
             </visual>
@@ -36,5 +36,5 @@
                         mash_filename="${back_cover_mash}"
                         scale_proportion="${scale_proportion}" />
-                <xacro:red_material/>
+                <xacro:set_material color="${back_cover_color}"/>
             </visual>
             <xacro:dummy_interia/>

File: simulation_ws/src/cr2_description/urdf/helpers/add_head.urdf.xacro (robot description, xacro)
@@ -19,5 +19,5 @@
                         mash_filename="${cr2_head_mash}"
                         scale_proportion="${scale_proportion}" />
-              <xacro:green_material/>
+              <xacro:set_material color="DarkGrey"/>
             </visual>
             <collision>

File: simulation_ws/src/cr2_description/urdf/materials.urdf.xacro (robot description, xacro)
@@ -31,3 +31,37 @@
     </material>
   </xacro:macro>
+  <xacro:macro name="set_material" params="color">
+  	<material name="${color}">
+	    <xacro:if value="${color == 'White'}">
+                <color rgba="1.0 1.0 1.0 1.0"/>
+	    </xacro:if>
+	    <xacro:if value="${color == 'Black'}">
+                <color rgba="0.0 0.0 0.0 1.0"/>
+	    </xacro:if>
+	    <xacro:if value="${color == 'Red'}">
+        	<color rgba="1.0 0.0 0.0 1.0"/>
+	    </xacro:if>
+	    <xacro:if value="${color == 'Green'}">
+        	<color rgba="0.0 1.0 0.0 1.0"/>
+	    </xacro:if>
+	    <xacro:if value="${color == 'Blue'}">
+                <color rgba="0.0 0.0 1.0 1.0"/>
+	    </xacro:if>
+	    <xacro:if value="${color == 'Yellow'}">
+                <color rgba="1.0 1.0 0.0 1.0"/>
+	    </xacro:if>
+	    <xacro:if value="${color == 'Grey'}">
+                <color rgba="0.5 0.5 0.5 1.0"/>
+	    </xacro:if>
+      <xacro:if value="${color == 'DarkGrey'}">
+                <color rgba="0.19 0.19 0.19 1.0"/>
+	    </xacro:if>
+    </material>
+  </xacro:macro>
+  <!-- Full list of colors is available here
+	  http://wiki.ros.org/simulator_gazebo/Tutorials/ListOfMaterials
+  -->
+  <xacro:macro name="set_gazebo_material" params="color">
+	  <material>Gazebo/${color}</material>
+  </xacro:macro>
 </robot>

Commit message: Added several tests

File: simulation_ws/src/cr2_description/params/cr2_params.urdf.xacro (robot description, xacro)
@@ -29,8 +29,10 @@
     <xacro:property name="tray_mash" value="package://cr2_description/meshes/tray.stl"/>
     <!--/MASHES-->
-    <!--DEBUG-->
-    <!--/DEBUG-->
-    <xacro:property name="body_color"           value="DarkGrey"/>
-    <xacro:property name="back_cover_color"     value="DarkGrey"/>
+    <xacro:property name="base_color"           value="DarkGrey"/>
+    <xacro:property name="body_color"           value="${base_color}"/>
+    <xacro:property name="back_cover_color"     value="${base_color}"/>
+    <xacro:property name="head_color"           value="${base_color}"/>
+    <xacro:property name="tray_color"           value="${base_color}"/>
+    <xacro:property name="monitor_color"           value="${base_color}"/>
 <!--BODY-->
     <!--TODO measure on assambled robot-->

File: simulation_ws/src/cr2_description/robot/cr2.gazebo.xacro (robot description, xacro)
@@ -39,5 +39,17 @@
   </gazebo>
   <gazebo reference="body">
-    <xacro:set_gazebo_material color="DarkGrey"/>
+    <xacro:set_gazebo_material color="${body_color}"/>
+  </gazebo>
+  <gazebo reference="head">
+    <xacro:set_gazebo_material color="${head_color}"/>
+  </gazebo>
+  <gazebo reference="tray">
+    <xacro:set_gazebo_material color="${tray_color}"/>
+  </gazebo>
+  <gazebo reference="monitor">
+    <xacro:set_gazebo_material color="${monitor_color}"/>
+  </gazebo>
+  <gazebo reference="back_cover">
+    <xacro:set_gazebo_material color="${back_cover_color}"/>
   </gazebo>
 <!--

File: simulation_ws/src/cr2_description/urdf/helpers/add_head.urdf.xacro (robot description, xacro)
@@ -19,5 +19,5 @@
                         mash_filename="${cr2_head_mash}"
                         scale_proportion="${scale_proportion}" />
-              <xacro:set_material color="DarkGrey"/>
+              <xacro:set_material color="${head_color}"/>
             </visual>
             <collision>
@@ -40,5 +40,5 @@
                         mash_filename="package://cr2_description/meshes/tray.stl"
                         scale_proportion="${scale_proportion}" />
-                <xacro:green_material/>
+                <xacro:set_material color="${tray_color}"/>
             </visual>
             <xacro:box_inertia
@@ -60,5 +60,5 @@
                       height="${monitor_height}"
                       depth="${monitor_lenght}"/>
-              <xacro:black_material/>
+              <xacro:set_material color="${monitor_color}"/>
             </visual>
             <xacro:box_inertia

File: simulation_ws/src/cr2_description/urdf/sensors/ultrasonic.urdf.xacro (robot description, xacro)
@@ -51,9 +51,9 @@
         </joint>
     </xacro:macro>
-    <xacro:macro name="ultrasonic_gazebo" params="position">
+  <xacro:macro name="ultrasonic_gazebo" params="position">
     <gazebo reference="ultrasonic_transmitter_oscillator_${position}_link">
       <material>Gazebo/Green</material>
       <sensor type="ray" name="sonar_${position}">
-        <pose>0 0 0 0 0 0</pose>
+      <pose>0 0 0 0 0 0</pose>
         <update_rate>1</update_rate>
         <visualize>false</visualize>
